Commit message: rename directory origin

File: catkin_ws/src/neo_simulation/worlds/small_warehouse.xacro (robot description, xacro)
@@ -25,8 +25,5 @@
         <collision name='collision'>
           <geometry>
-            <mesh>
-              <uri>model://aws_robomaker_warehouse_ShelfF_01/meshes/aws_robomaker_warehouse_ShelfF_01_collision.DAE</uri>
-              <scale>1 1 1</scale>
-            </mesh>
+            <mesh filename="package://neo_simulation/models/aws_robomaker_warehouse_ShelfF_01/meshes/aws_robomaker_warehouse_ShelfF_01_collision.DAE" <scale>1 1 1</scale>
           </geometry>
           <surface>
@@ -52,7 +49,5 @@
         <visual name='visual'>
           <geometry>
-            <mesh>
-              <uri>model://aws_robomaker_warehouse_ShelfF_01/meshes/aws_robomaker_warehouse_ShelfF_01_visual.DAE</uri>
-            </mesh>
+            <mesh filename="package://neo_simulation/models/aws_robomaker_warehouse_ShelfF_01/meshes/aws_robomaker_warehouse_ShelfF_01_visual.DAE"/>
           </geometry>
           <meta>
@@ -86,7 +81,5 @@
         <collision name='collision'>
           <geometry>
-            <mesh>
-              <uri>model://aws_robomaker_warehouse_WallB_01/meshes/aws_robomaker_warehouse_WallB_01_collision.DAE</uri>
-              <scale>1 1 1</scale>
+            <mesh filename="package://neo_simulation/models/aws_robomaker_warehouse_WallB_01/meshes/aws_robomaker_warehouse_WallB_01_collision.DAE" <scale>1 1 1</scale>
             </mesh>
           </geometry>
@@ -113,7 +106,5 @@
         <visual name='visual'>
           <geometry>
-            <mesh>
-              <uri>model://aws_robomaker_warehouse_WallB_01/meshes/aws_robomaker_warehouse_WallB_01_visual.DAE</uri>
-            </mesh>
+            <mesh filename="package://neo_simulation/models/aws_robomaker_warehouse_WallB_01/meshes/aws_robomaker_warehouse_WallB_01_visual.DAE"/>
           </geometry>
           <meta>
@@ -147,8 +138,5 @@
         <collision name='collision'>
           <geometry>
-            <mesh>
-              <uri>model://aws_robomaker_warehouse_ShelfE_01/meshes/aws_robomaker_warehouse_ShelfE_01_collision.DAE</uri>
-              <scale>1 1 1</scale>
-            </mesh>
+            <mesh filename="package://neo_simulation/models/aws_robomaker_warehouse_ShelfE_01/meshes/aws_robomaker_warehouse_ShelfE_01_collision.DAE" <scale>1 1 1</scale>
           </geometry>
           <surface>
@@ -174,7 +162,5 @@
         <visual name='visual'>
           <geometry>
-            <mesh>
-              <uri>model://aws_robomaker_warehouse_ShelfE_01/meshes/aws_robomaker_warehouse_ShelfE_01_visual.DAE</uri>
-            </mesh>
+            <mesh filename="package://neo_simulation/models/aws_robomaker_warehouse_ShelfE_01/meshes/aws_robomaker_warehouse_ShelfE_01_visual.DAE"/>
           </geometry>
           <meta>
@@ -208,8 +194,5 @@
         <collision name='collision'>
           <geometry>
-            <mesh>
-              <uri>model://aws_robomaker_warehouse_ShelfE_01/meshes/aws_robomaker_warehouse_ShelfE_01_collision.DAE</uri>
-              <scale>1 1 1</scale>
-            </mesh>
+            <mesh filename="package://neo_simulation/models/aws_robomaker_warehouse_ShelfE_01/meshes/aws_robomaker_warehouse_ShelfE_01_collision.DAE" <scale>1 1 1</scale>
           </geometry>
           <surface>
@@ -235,7 +218,5 @@
         <visual name='visual'>
           <geometry>
-            <mesh>
-              <uri>model://aws_robomaker_warehouse_ShelfE_01/meshes/aws_robomaker_warehouse_ShelfE_01_visual.DAE</uri>
-            </mesh>
+            <mesh filename="package://neo_simulation/models/aws_robomaker_warehouse_ShelfE_01/meshes/aws_robomaker_warehouse_ShelfE_01_visual.DAE"/>
           </geometry>
           <meta>
@@ -269,8 +250,5 @@
         <collision name='collision'>
           <geometry>
-            <mesh>
-              <uri>model://aws_robomaker_warehouse_ShelfE_01/meshes/aws_robomaker_warehouse_ShelfE_01_collision.DAE</uri>
-              <scale>1 1 1</scale>
-            </mesh>
+            <mesh filename="package://neo_simulation/models/aws_robomaker_warehouse_ShelfE_01/meshes/aws_robomaker_warehouse_ShelfE_01_collision.DAE" <scale>1 1 1</scale>
           </geometry>
           <surface>
@@ -296,7 +274,5 @@
         <visual name='visual'>
           <geometry>
-            <mesh>
-              <uri>model://aws_robomaker_warehouse_ShelfE_01/meshes/aws_robomaker_warehouse_ShelfE_01_visual.DAE</uri>
-            </mesh>
+            <mesh filename="package://neo_simulation/models/aws_robomaker_warehouse_ShelfE_01/meshes/aws_robomaker_warehouse_ShelfE_01_visual.DAE"/>
           </geometry>
           <meta>
@@ -330,8 +306,5 @@
         <collision name='collision'>
           <geometry>
-            <mesh>
-              <uri>model://aws_robomaker_warehouse_ShelfD_01/meshes/aws_robomaker_warehouse_ShelfD_01_collision.DAE</uri>
-              <scale>1 1 1</scale>
-            </mesh>
+            <mesh filename="package://neo_simulation/models/aws_robomaker_warehouse_ShelfD_01/meshes/aws_robomaker_warehouse_ShelfD_01_collision.DAE" <scale>1 1 1</scale>
           </geometry>
           <surface>
@@ -357,7 +330,5 @@
         <visual name='visual'>
           <geometry>
-            <mesh>
-              <uri>model://aws_robomaker_warehouse_ShelfD_01/meshes/aws_robomaker_warehouse_ShelfD_01_visual.DAE</uri>
-            </mesh>
+            <mesh filename="package://neo_simulation/models/aws_robomaker_warehouse_ShelfD_01/meshes/aws_robomaker_warehouse_ShelfD_01_visual.DAE"/>
           </geometry>
           <meta>
@@ -391,8 +362,5 @@
         <collision name='collision'>
           <geometry>
-            <mesh>
-              <uri>model://aws_robomaker_warehouse_ShelfD_01/meshes/aws_robomaker_warehouse_ShelfD_01_collision.DAE</uri>
-              <scale>1 1 1</scale>
-            </mesh>
+            <mesh filename="package://neo_simulation/models/aws_robomaker_warehouse_ShelfD_01/meshes/aws_robomaker_warehouse_ShelfD_01_collision.DAE" <scale>1 1 1</scale>
           </geometry>
           <surface>
@@ -418,7 +386,5 @@
         <visual name='visual'>
           <geometry>
-            <mesh>
-              <uri>model://aws_robomaker_warehouse_ShelfD_01/meshes/aws_robomaker_warehouse_ShelfD_01_visual.DAE</uri>
-            </mesh>
+            <mesh filename="package://neo_simulation/models/aws_robomaker_warehouse_ShelfD_01/meshes/aws_robomaker_warehouse_ShelfD_01_visual.DAE"/>
           </geometry>
           <meta>
@@ -452,8 +418,5 @@
         <collision name='collision'>
           <geometry>
-            <mesh>
-              <uri>model://aws_robomaker_warehouse_ShelfD_01/meshes/aws_robomaker_warehouse_ShelfD_01_collision.DAE</uri>
-              <scale>1 1 1</scale>
-            </mesh>
+            <mesh filename="package://neo_simulation/models/aws_robomaker_warehouse_ShelfD_01/meshes/aws_robomaker_warehouse_ShelfD_01_collision.DAE" <scale>1 1 1</scale>
           </geometry>
           <surface>
@@ -479,7 +442,5 @@
         <visual name='visual'>
           <geometry>
-            <mesh>
-              <uri>model://aws_robomaker_warehouse_ShelfD_01/meshes/aws_robomaker_warehouse_ShelfD_01_visual.DAE</uri>
-            </mesh>
+            <mesh filename="package://neo_simulation/models/aws_robomaker_warehouse_ShelfD_01/meshes/aws_robomaker_warehouse_ShelfD_01_visual.DAE"/>
           </geometry>
           <meta>
@@ -513,8 +474,5 @@
         <collision name='collision'>
           <geometry>
-            <mesh>
-              <uri>model://aws_robomaker_warehouse_GroundB_01/meshes/aws_robomaker_warehouse_GroundB_01_collision.DAE</uri>
-              <scale>1 1 1</scale>
-            </mesh>
+            <mesh filename="package://neo_simulation/models/aws_robomaker_warehouse_GroundB_01/meshes/aws_robomaker_warehouse_GroundB_01_collision.DAE" <scale>1 1 1</scale>
           </geometry>
           <surface>
@@ -540,7 +498,5 @@
         <visual name='visual'>
           <geometry>
-            <mesh>
-              <uri>model://aws_robomaker_warehouse_GroundB_01/meshes/aws_robomaker_warehouse_GroundB_01_visual.DAE</uri>
-            </mesh>
+            <mesh filename="package://neo_simulation/models/aws_robomaker_warehouse_GroundB_01/meshes/aws_robomaker_warehouse_GroundB_01_visual.DAE"/>
           </geometry>
           <meta>
@@ -574,8 +530,5 @@
         <collision name='collision'>
           <geometry>
-            <mesh>
-              <uri>model://aws_robomaker_warehouse_Lamp_01/meshes/aws_robomaker_warehouse_Lamp_01_collision.DAE</uri>
-              <scale>1 1 1</scale>
-            </mesh>
+            <mesh filename="package://neo_simulation/models/aws_robomaker_warehouse_Lamp_01/meshes/aws_robomaker_warehouse_Lamp_01_collision.DAE" <scale>1 1 1</scale>
           </geometry>
           <surface>
@@ -601,7 +554,5 @@
         <visual name='visual'>
           <geometry>
-            <mesh>
-              <uri>model://aws_robomaker_warehouse_Lamp_01/meshes/aws_robomaker_warehouse_Lamp_01_visual.DAE</uri>
-            </mesh>
+            <mesh filename="package://neo_simulation/models/aws_robomaker_warehouse_Lamp_01/meshes/aws_robomaker_warehouse_Lamp_01_visual.DAE"/>
           </geometry>
           <meta>
@@ -640,7 +591,5 @@
         <visual name='visual'>
           <geometry>
-            <mesh>
-              <uri>model://aws_robomaker_warehouse_Bucket_01/meshes/aws_robomaker_warehouse_Bucket_01_visual.DAE</uri>
-            </mesh>
+            <mesh filename="package://neo_simulation/models/aws_robomaker_warehouse_Bucket_01/meshes/aws_robomaker_warehouse_Bucket_01_visual.DAE"/>
           </geometry>
           <meta>
@@ -653,8 +602,5 @@
           <pose>0 0 0 0 -0 0</pose>
           <geometry>
-            <mesh>
-              <uri>model://aws_robomaker_warehouse_Bucket_01/meshes/aws_robomaker_warehouse_Bucket_01_collision.DAE</uri>
-              <scale>1 1 1</scale>
-            </mesh>
+            <mesh filename="package://neo_simulation/models/aws_robomaker_warehouse_Bucket_01/meshes/aws_robomaker_warehouse_Bucket_01_collision.DAE"/>
           </geometry>
           <surface>
@@ -711,7 +657,5 @@
         <visual name='visual'>
           <geometry>
-            <mesh>
-              <uri>model://aws_robomaker_warehouse_Bucket_01/meshes/aws_robomaker_warehouse_Bucket_01_visual.DAE</uri>
-            </mesh>
+            <mesh filename="package://neo_simulation/models/aws_robomaker_warehouse_Bucket_01/meshes/aws_robomaker_warehouse_Bucket_01_visual.DAE"/>
           </geometry>
           <meta>
@@ -724,8 +668,5 @@
           <pose>0 0 0 0 -0 0</pose>
           <geometry>
-            <mesh>
-              <uri>model://aws_robomaker_warehouse_Bucket_01/meshes/aws_robomaker_warehouse_Bucket_01_collision.DAE</uri>
-              <scale>1 1 1</scale>
-            </mesh>
+            <mesh filename="package://neo_simulation/models/aws_robomaker_warehouse_Bucket_01/meshes/aws_robomaker_warehouse_Bucket_01_collision.DAE"/>
           </geometry>
           <surface>
@@ -782,7 +723,5 @@
         <visual name='visual'>
           <geometry>
-            <mesh>
-              <uri>model://aws_robomaker_warehouse_Bucket_01/meshes/aws_robomaker_warehouse_Bucket_01_visual.DAE</uri>
-            </mesh>
+            <mesh filename="package://neo_simulation/models/aws_robomaker_warehouse_Bucket_01/meshes/aws_robomaker_warehouse_Bucket_01_visual.DAE"/>
           </geometry>
           <meta>
@@ -795,8 +734,5 @@
           <pose>0 0 0 0 -0 0</pose>
           <geometry>
-            <mesh>
-              <uri>model://aws_robomaker_warehouse_Bucket_01/meshes/aws_robomaker_warehouse_Bucket_01_collision.DAE</uri>
-              <scale>1 1 1</scale>
-            </mesh>
+            <mesh filename="package://neo_simulation/models/aws_robomaker_warehouse_Bucket_01/meshes/aws_robomaker_warehouse_Bucket_01_collision.DAE"/>
           </geometry>
           <surface>
@@ -848,8 +784,5 @@
         <collision name='collision'>
           <geometry>
-            <mesh>
-              <uri>model://aws_robomaker_warehouse_ClutteringA_01/meshes/aws_robomaker_warehouse_ClutteringA_01_collision.DAE</uri>
-              <scale>1 1 1</scale>
-            </mesh>
+            <mesh filename="package://neo_simulation/models/aws_robomaker_warehouse_ClutteringA_01/meshes/aws_robomaker_warehouse_ClutteringA_01_collision.DAE"/>
           </geometry>
           <surface>
@@ -881,7 +814,5 @@
         <visual name='visual'>
           <geometry>
-            <mesh>
-              <uri>model://aws_robomaker_warehouse_ClutteringA_01/meshes/aws_robomaker_warehouse_ClutteringA_01_visual.DAE</uri>
-            </mesh>
+            <mesh filename="package://neo_simulation/models/aws_robomaker_warehouse_ClutteringA_01/meshes/aws_robomaker_warehouse_ClutteringA_01_visual.DAE"/>
           </geometry>
           <meta>
@@ -915,8 +846,5 @@
         <collision name='collision'>
           <geometry>
-            <mesh>
-              <uri>model://aws_robomaker_warehouse_ClutteringA_01/meshes/aws_robomaker_warehouse_ClutteringA_01_collision.DAE</uri>
-              <scale>1 1 1</scale>
-            </mesh>
+            <mesh filename="package://neo_simulation/models/aws_robomaker_warehouse_ClutteringA_01/meshes/aws_robomaker_warehouse_ClutteringA_01_collision.DAE"/>
           </geometry>
           <surface>
@@ -948,7 +876,5 @@
         <visual name='visual'>
           <geometry>
-            <mesh>
-              <uri>model://aws_robomaker_warehouse_ClutteringA_01/meshes/aws_robomaker_warehouse_ClutteringA_01_visual.DAE</uri>
-            </mesh>
+            <mesh filename="package://neo_simulation/models/aws_robomaker_warehouse_ClutteringA_01/meshes/aws_robomaker_warehouse_ClutteringA_01_visual.DAE"/>
           </geometry>
           <meta>
@@ -982,8 +908,5 @@
         <collision name='collision'>
           <geometry>
-            <mesh>
-              <uri>model://aws_robomaker_warehouse_ClutteringA_01/meshes/aws_robomaker_warehouse_ClutteringA_01_collision.DAE</uri>
-              <scale>1 1 1</scale>
-            </mesh>
+            <mesh filename="package://neo_simulation/models/aws_robomaker_warehouse_ClutteringA_01/meshes/aws_robomaker_warehouse_ClutteringA_01_collision.DAE"/>
           </geometry>
           <surface>
@@ -1015,7 +938,5 @@
         <visual name='visual'>
           <geometry>
-            <mesh>
-              <uri>model://aws_robomaker_warehouse_ClutteringA_01/meshes/aws_robomaker_warehouse_ClutteringA_01_visual.DAE</uri>
-            </mesh>
+            <mesh filename="package://neo_simulation/models/aws_robomaker_warehouse_ClutteringA_01/meshes/aws_robomaker_warehouse_ClutteringA_01_visual.DAE"/>
           </geometry>
           <meta>
@@ -1049,8 +970,5 @@
         <collision name='collision'>
           <geometry>
-            <mesh>
-              <uri>model://aws_robomaker_warehouse_ClutteringC_01/meshes/aws_robomaker_warehouse_ClutteringC_01_collision.DAE</uri>
-              <scale>1 1 1</scale>
-            </mesh>
+            <mesh filename="package://neo_simulation/models/aws_robomaker_warehouse_ClutteringC_01/meshes/aws_robomaker_warehouse_ClutteringC_01_collision.DAE"/>
           </geometry>
           <surface>
@@ -1082,7 +1000,5 @@
         <visual name='visual'>
           <geometry>
-            <mesh>
-              <uri>model://aws_robomaker_warehouse_ClutteringC_01/meshes/aws_robomaker_warehouse_ClutteringC_01_visual.DAE</uri>
-            </mesh>
+            <mesh filename="package://neo_simulation/models/aws_robomaker_warehouse_ClutteringC_01/meshes/aws_robomaker_warehouse_ClutteringC_01_visual.DAE"/>
           </geometry>
           <meta>
@@ -1116,8 +1032,5 @@
         <collision name='collision'>
           <geometry>
-            <mesh>
-              <uri>model://aws_robomaker_warehouse_ClutteringC_01/meshes/aws_robomaker_warehouse_ClutteringC_01_collision.DAE</uri>
-              <scale>1 1 1</scale>
-            </mesh>
+            <mesh filename="package://neo_simulation/models/aws_robomaker_warehouse_ClutteringC_01/meshes/aws_robomaker_warehouse_ClutteringC_01_collision.DAE"/>
           </geometry>
           <surface>
@@ -1149,7 +1062,5 @@
         <visual name='visual'>
           <geometry>
-            <mesh>
-              <uri>model://aws_robomaker_warehouse_ClutteringC_01/meshes/aws_robomaker_warehouse_ClutteringC_01_visual.DAE</uri>
-            </mesh>
+            <mesh filename="package://neo_simulation/models/aws_robomaker_warehouse_ClutteringC_01/meshes/aws_robomaker_warehouse_ClutteringC_01_visual.DAE"/>
           </geometry>
           <meta>
@@ -1183,8 +1094,5 @@
         <collision name='collision'>
           <geometry>
-            <mesh>
-              <uri>model://aws_robomaker_warehouse_ClutteringC_01/meshes/aws_robomaker_warehouse_ClutteringC_01_collision.DAE</uri>
-              <scale>1 1 1</scale>
-            </mesh>
+            <mesh filename="package://neo_simulation/models/aws_robomaker_warehouse_ClutteringC_01/meshes/aws_robomaker_warehouse_ClutteringC_01_collision.DAE"/>
           </geometry>
           <surface>
@@ -1216,7 +1124,5 @@
         <visual name='visual'>
           <geometry>
-            <mesh>
-              <uri>model://aws_robomaker_warehouse_ClutteringC_01/meshes/aws_robomaker_warehouse_ClutteringC_01_visual.DAE</uri>
-            </mesh>
+            <mesh filename="package://neo_simulation/models/aws_robomaker_warehouse_ClutteringC_01/meshes/aws_robomaker_warehouse_ClutteringC_01_visual.DAE"/>
           </geometry>
           <meta>
@@ -1250,8 +1156,5 @@
         <collision name='collision'>
           <geometry>
-            <mesh>
-              <uri>model://aws_robomaker_warehouse_ClutteringC_01/meshes/aws_robomaker_warehouse_ClutteringC_01_collision.DAE</uri>
-              <scale>1 1 1</scale>
-            </mesh>
+            <mesh filename="package://neo_simulation/models/aws_robomaker_warehouse_ClutteringC_01/meshes/aws_robomaker_warehouse_ClutteringC_01_collision.DAE"/>
           </geometry>
           <surface>
@@ -1283,7 +1186,5 @@
         <visual name='visual'>
           <geometry>
-            <mesh>
-              <uri>model://aws_robomaker_warehouse_ClutteringC_01/meshes/aws_robomaker_warehouse_ClutteringC_01_visual.DAE</uri>
-            </mesh>
+            <mesh filename="package://neo_simulation/models/aws_robomaker_warehouse_ClutteringC_01/meshes/aws_robomaker_warehouse_ClutteringC_01_visual.DAE"/>
           </geometry>
           <meta>
@@ -1317,8 +1218,5 @@
         <collision name='collision'>
           <geometry>
-            <mesh>
-              <uri>model://aws_robomaker_warehouse_ClutteringC_01/meshes/aws_robomaker_warehouse_ClutteringC_01_collision.DAE</uri>
-              <scale>1 1 1</scale>
-            </mesh>
+            <mesh filename="package://neo_simulation/models/aws_robomaker_warehouse_ClutteringC_01/meshes/aws_robomaker_warehouse_ClutteringC_01_collision.DAE"/>
           </geometry>
           <surface>
@@ -1350,7 +1248,5 @@
         <visual name='visual'>
           <geometry>
-            <mesh>
-              <uri>model://aws_robomaker_warehouse_ClutteringC_01/meshes/aws_robomaker_warehouse_ClutteringC_01_visual.DAE</uri>
-            </mesh>
+            <mesh filename="package://neo_simulation/models/aws_robomaker_warehouse_ClutteringC_01/meshes/aws_robomaker_warehouse_ClutteringC_01_visual.DAE"/>
           </geometry>
           <meta>
@@ -1384,8 +1280,5 @@
         <collision name='collision'>
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