Commit message: remove mpo_500_

File: catkin_ws/src/neo_simulation/robots/mpo_500/mpo_500.urdf.xacro (robot description, xacro)
@@ -2,13 +2,13 @@
 <robot name="mpo_500" xmlns:xacro="http://www.ros.org/wiki/xacro">
   <!--GAZEBO REFERENCES -->
-  <xacro:include filename="$(find neo_simulation)/robots/mpo_500/xacros/mpo_500_gazebo.xacro" />
+  <xacro:include filename="$(find neo_simulation)/robots/xacros/gazebo.xacro" />
   <!-- BODY -->
-  <xacro:include filename="$(find neo_simulation)/robots/mpo_500/xacros/mpo_500_body.xacro" />
+  <xacro:include filename="$(find neo_simulation)/robots/xacros/body.xacro" />
   <!-- WHEELS -->
-  <xacro:include filename="$(find neo_simulation)/robots/mpo_500/xacros/omni_wheel.xacro" />
+  <xacro:include filename="$(find neo_simulation)/robots/xacros/omni_wheel.xacro" />
   <!-- SENSORS -->
   <!-- <xacro:include filename="$(find neo_simulation)/robots/mpo_500/xacros/sick_S300.xacro" /> -->
   <!-- Microscan - Comment/Uncomment if required -->
-  <xacro:include filename="$(find neo_simulation)/robots/mpo_500/xacros/micro_scan.xacro" />
+  <xacro:include filename="$(find neo_simulation)/robots/xacros/micro_scan.xacro" />
   <!--Ultrasonics, cameras and IMU's  -->
   <!-->
@@ -19,18 +19,18 @@
   <link name="base_link" />
   <!-- Base link macro -->
-  <xacro:mpo_500_base name="base_footprint" parent="base_link">
+  <xacro:base name="base_footprint" parent="base_link">
     <origin xyz="0 0 0" rpy="0 0 0" />
-  </xacro:mpo_500_base>
+  </xacro:base>
   <!-- Wheel Macro -->
-  <xacro:omni_wheel_250 name="mpo_500_omni_wheel_front_left" parent="base_footprint">
+  <xacro:omni_wheel_250 name="omni_wheel_front_left" parent="base_footprint">
     <origin xyz="0.25 0.28 0.13" rpy="0 0 0" />
   </xacro:omni_wheel_250>
-  <xacro:omni_wheel_250 name="mpo_500_omni_wheel_front_right" parent="base_footprint">
+  <xacro:omni_wheel_250 name="omni_wheel_front_right" parent="base_footprint">
     <origin xyz="0.25 -0.28 0.13" rpy="0 0 3.14" />
   </xacro:omni_wheel_250>
-  <xacro:omni_wheel_250 name="mpo_500_omni_wheel_back_left" parent="base_footprint">
+  <xacro:omni_wheel_250 name="omni_wheel_back_left" parent="base_footprint">
     <origin xyz="-0.25 0.28 0.13" rpy="0 0 0" />
   </xacro:omni_wheel_250>
-  <xacro:omni_wheel_250 name="mpo_500_omni_wheel_back_right" parent="base_footprint">
+  <xacro:omni_wheel_250 name="omni_wheel_back_right" parent="base_footprint">
     <origin xyz="-0.25 -0.28 0.13" rpy="0 0 3.14" />
   </xacro:omni_wheel_250>
@@ -121,37 +121,37 @@
     <origin xyz="0 0 0.38" rpy="0 0 0" />
   </xacro:camera> -->
-  <transmission name="mpo_500_omni_wheel_front_left">
+  <transmission name="omni_wheel_front_left">
     <type>transmission_interface/SimpleTransmission</type>
-    <joint name="mpo_500_omni_wheel_front_left_joint">
+    <joint name="omni_wheel_front_left_joint">
       <hardwareInterface>hardware_interface/VelocityJointInterface</hardwareInterface>
     </joint>
-    <actuator name="mpo_500_omni_wheel_front_left_motor">
+    <actuator name="omni_wheel_front_left_motor">
       <mechanicalReduction>1</mechanicalReduction>
     </actuator>
   </transmission>
-  <transmission name="mpo_500_omni_wheel_front_right">
+  <transmission name="omni_wheel_front_right">
     <type>transmission_interface/SimpleTransmission</type>
-    <joint name="mpo_500_omni_wheel_front_right_joint">
+    <joint name="omni_wheel_front_right_joint">
       <hardwareInterface>hardware_interface/VelocityJointInterface</hardwareInterface>
     </joint>
-    <actuator name="mpo_500_omni_wheel_front_right_motor">
+    <actuator name="omni_wheel_front_right_motor">
       <mechanicalReduction>1</mechanicalReduction>
     </actuator>
   </transmission>
-  <transmission name="mpo_500_omni_wheel_back_left">
+  <transmission name="omni_wheel_back_left">
     <type>transmission_interface/SimpleTransmission</type>
-    <joint name="mpo_500_omni_wheel_back_left_joint">
+    <joint name="omni_wheel_back_left_joint">
       <hardwareInterface>hardware_interface/VelocityJointInterface</hardwareInterface>
     </joint>
-    <actuator name="mpo_500_omni_wheel_back_left_motor">
+    <actuator name="omni_wheel_back_left_motor">
       <mechanicalReduction>1</mechanicalReduction>
     </actuator>
   </transmission>
-  <transmission name="mpo_500_omni_wheel_back_right">
+  <transmission name="omni_wheel_back_right">
     <type>transmission_interface/SimpleTransmission</type>
-    <joint name="mpo_500_omni_wheel_back_right_joint">
+    <joint name="omni_wheel_back_right_joint">
       <hardwareInterface>hardware_interface/VelocityJointInterface</hardwareInterface>
     </joint>
-    <actuator name="mpo_500_omni_wheel_back_right_motor">
+    <actuator name="omni_wheel_back_right_motor">
       <mechanicalReduction>1</mechanicalReduction>
     </actuator>

File: catkin_ws/src/neo_simulation/robots/xacros/body.xacro (robot description, xacro)
@@ -1,5 +1,5 @@
 <?xml version="1.0"?>
 <robot xmlns:xacro="http://www.ros.org/wiki/xacro" name="mpo_500">
-  <xacro:macro name="mpo_500_base" params="name parent *origin">
+  <xacro:macro name="base" params="name parent *origin">
     <joint name="${name}_joint" type="fixed">
       <xacro:insert_block name="origin" />

File: catkin_ws/src/neo_simulation/robots/xacros/gazebo.xacro (robot description, xacro)
@@ -171,5 +171,5 @@
 </gazebo>
 <gazebo>
-    <plugin name="mpo_500_controller" filename="libgazebo_ros_planar_move.so">
+    <plugin name="controller" filename="libgazebo_ros_planar_move.so">
       <commandTopic>cmd_vel</commandTopic>
       <odometryTopic>odom</odometryTopic>
