Commit message: remove mpo_500 reference

File: catkin_ws/src/neo_simulation/robots/xacros/body.xacro (robot description, xacro)
@@ -21,5 +21,5 @@
         <origin xyz="0. 0. 0" rpy="-1.571 0 1.571" />
         <geometry>
-            <mesh filename="package://neo_simulation/robots/mpo_500/meshes/MPO-500-BODY.dae" scale="0.001 0.001 0.001"/>
+            <mesh filename="package://neo_simulation/robots/meshes/MPO-500-BODY.dae" scale="0.001 0.001 0.001"/>
         </geometry>
       </visual>
@@ -28,5 +28,5 @@
         <geometry>
           <!--<box size="0.68 0.41 0.25"/> -->
-           <mesh filename="package://neo_simulation/robots/mpo_500/meshes/MPO-500-BODY.dae" scale="0.001 0.001 0.001"/>
+           <mesh filename="package://neo_simulation/robots/meshes/MPO-500-BODY.dae" scale="0.001 0.001 0.001"/>
         </geometry>
       </collision>

File: catkin_ws/src/neo_simulation/robots/xacros/micro_scan.xacro (robot description, xacro)
@@ -17,5 +17,5 @@
         <origin xyz="0 0 -0.06" rpy="1.57 0 0" />
       <geometry>
-        <mesh filename="package://neo_simulation/robots/mpo_500/meshes/SICK-MICROSCAN3.dae" scale="0.001 0.001 0.001" />
+        <mesh filename="package://neo_simulation/robots/meshes/SICK-MICROSCAN3.dae" scale="0.001 0.001 0.001" />
         </geometry>
       </visual>
@@ -23,5 +23,5 @@
         <origin xyz="0 0 -0.06" rpy="1.57 0 0" />
         <geometry>
-          <mesh filename="package://neo_simulation/robots/mpo_500/meshes/SICK-MICROSCAN3.dae" scale="0.001 0.001 0.001" />
+          <mesh filename="package://neo_simulation/robots/meshes/SICK-MICROSCAN3.dae" scale="0.001 0.001 0.001" />
         </geometry>
       </collision>

File: catkin_ws/src/neo_simulation/robots/xacros/omni_wheel.xacro (robot description, xacro)
@@ -22,5 +22,5 @@
      <origin xyz="0 0 0" rpy="0 0 0"/>
      <geometry>
-        <mesh filename="package://neo_simulation/robots/mpo_500/meshes/MPO-500-WHEEL.dae" scale="0.001 0.001 0.001"/>
+        <mesh filename="package://neo_simulation/robots/meshes/MPO-500-WHEEL.dae" scale="0.001 0.001 0.001"/>
      </geometry>
     </visual>
@@ -28,5 +28,5 @@
      <origin xyz="0 0 0" rpy="0 1.57 1.57" />
      <geometry>
-        <!-- <mesh filename="package://neo_simulation/robots/mpo_500/meshes/MPO-500-WHEEL.dae" scale="0.001 0.001 0.001"/> -->
+        <!-- <mesh filename="package://neo_simulation/robots/meshes/MPO-500-WHEEL.dae" scale="0.001 0.001 0.001"/> -->
        <!-- <cylinder radius="0.126" length="0.110"/> -->
       <sphere radius="0.117" />

File: catkin_ws/src/neo_simulation/robots/xacros/sick_S300.xacro (robot description, xacro)
@@ -17,5 +17,5 @@
         <origin xyz="0 0 -0.12" rpy="-1.57 0 3.14" />
         <geometry>
-        <mesh filename="package://neo_simulation/robots/mpo_500/meshes/SICK-S300.dae" scale="0.001 0.001 0.001" />
+        <mesh filename="package://neo_simulation/robots/meshes/SICK-S300.dae" scale="0.001 0.001 0.001" />
         </geometry>
       </visual>
@@ -23,5 +23,5 @@
         <origin xyz="0 0 -0.12" rpy="-1.57 0 3.14" />
         <geometry>
-        <mesh filename="package://neo_simulation/robots/mpo_500/meshes/SICK-S300.dae" scale="0.001 0.001 0.001" />
+        <mesh filename="package://neo_simulation/robots/meshes/SICK-S300.dae" scale="0.001 0.001 0.001" />
         </geometry>
       </collision>

File: catkin_ws/src/neo_simulation/robots/xacros/sick_laser.xacro (robot description, xacro)
@@ -18,5 +18,5 @@
       <origin xyz="0 0 -0.12" rpy="-1.57 0 3.14" />
         <geometry>
-        <mesh filename="package://neo_simulation/robots/mpo_500/meshes/SICK-S300.dae" scale="0.001 0.001 0.001" />
+        <mesh filename="package://neo_simulation/robots/meshes/SICK-S300.dae" scale="0.001 0.001 0.001" />
         </geometry>
       </visual>
@@ -24,5 +24,5 @@
         <origin xyz="0 0 0" rpy="-1.57 0 3.14" />
         <geometry>
-        <mesh filename="package://neo_simulation/robots/mpo_500/meshes/SICK-S300.dae" scale="0.001 0.001 0.001" />
+        <mesh filename="package://neo_simulation/robots/meshes/SICK-S300.dae" scale="0.001 0.001 0.001" />
         </geometry>
       </collision>
@@ -30,5 +30,5 @@
 <!--  <origin xyz="-0.0 0 -0.06" rpy="1.57 0 0" />
       <geometry>
-      <mesh filename="package://neo_simulation/robots/mpo_500/meshes/SICK-MICROSCAN3.dae" scale="0.001 0.001 0.001" />
+      <mesh filename="package://neo_simulation/robots/meshes/SICK-MICROSCAN3.dae" scale="0.001 0.001 0.001" />
       </geometry>
       </visual>
@@ -36,5 +36,5 @@
  <origin xyz="-0.0 0 -0.06" rpy="1.57 0 0" />
       <geometry>
-        <mesh filename="package://neo_simulation/robots/mp_500/meshes/SICK-MICROSCAN3.dae" scale="0.001 0.001 0.001" />
+        <mesh filename="package://neo_simulation/robots/meshes/SICK-MICROSCAN3.dae" scale="0.001 0.001 0.001" />
         </geometry>
       </collision> -->
