Commit message: rename neo_simulation to robot_nav

File: catkin_ws/src/robot_nav/robots/robot.urdf.xacro (robot description, xacro)
@@ -2,13 +2,13 @@
 <robot name="mpo_500" xmlns:xacro="http://www.ros.org/wiki/xacro">
   <!--GAZEBO REFERENCES -->
-  <xacro:include filename="$(find neo_simulation)/robots/xacros/gazebo.xacro" />
+  <xacro:include filename="$(find robot_nav)/robots/xacros/gazebo.xacro" />
   <!-- BODY -->
-  <xacro:include filename="$(find neo_simulation)/robots/xacros/body.xacro" />
+  <xacro:include filename="$(find robot_nav)/robots/xacros/body.xacro" />
   <!-- WHEELS -->
-  <xacro:include filename="$(find neo_simulation)/robots/xacros/omni_wheel.xacro" />
+  <xacro:include filename="$(find robot_nav)/robots/xacros/omni_wheel.xacro" />
   <!-- SENSORS -->
-  <!-- <xacro:include filename="$(find neo_simulation)/robots/xacros/sick_S300.xacro" /> -->
+  <!-- <xacro:include filename="$(find robot_nav)/robots/xacros/sick_S300.xacro" /> -->
   <!-- Microscan - Comment/Uncomment if required -->
-  <xacro:include filename="$(find neo_simulation)/robots/xacros/micro_scan.xacro" />
+  <xacro:include filename="$(find robot_nav)/robots/xacros/micro_scan.xacro" />
   <link name="base_link" />
   <!-- Base link macro -->

File: catkin_ws/src/robot_nav/robots/xacros/body.xacro (robot description, xacro)
@@ -21,5 +21,5 @@
         <origin xyz="0. 0. 0" rpy="-1.571 0 1.571" />
         <geometry>
-            <mesh filename="package://neo_simulation/robots/meshes/MPO-500-BODY.dae" scale="0.001 0.001 0.001"/>
+            <mesh filename="package://robot_nav/robots/meshes/MPO-500-BODY.dae" scale="0.001 0.001 0.001"/>
         </geometry>
       </visual>
@@ -28,5 +28,5 @@
         <geometry>
           <!--<box size="0.68 0.41 0.25"/> -->
-           <mesh filename="package://neo_simulation/robots/meshes/MPO-500-BODY.dae" scale="0.001 0.001 0.001"/>
+           <mesh filename="package://robot_nav/robots/meshes/MPO-500-BODY.dae" scale="0.001 0.001 0.001"/>
         </geometry>
       </collision>

File: catkin_ws/src/robot_nav/robots/xacros/micro_scan.xacro (robot description, xacro)
@@ -17,5 +17,5 @@
         <origin xyz="0 0 -0.06" rpy="1.57 0 0" />
       <geometry>
-        <mesh filename="package://neo_simulation/robots/meshes/SICK-MICROSCAN3.dae" scale="0.001 0.001 0.001" />
+        <mesh filename="package://robot_nav/robots/meshes/SICK-MICROSCAN3.dae" scale="0.001 0.001 0.001" />
         </geometry>
       </visual>
@@ -23,5 +23,5 @@
         <origin xyz="0 0 -0.06" rpy="1.57 0 0" />
         <geometry>
-          <mesh filename="package://neo_simulation/robots/meshes/SICK-MICROSCAN3.dae" scale="0.001 0.001 0.001" />
+          <mesh filename="package://robot_nav/robots/meshes/SICK-MICROSCAN3.dae" scale="0.001 0.001 0.001" />
         </geometry>
       </collision>

File: catkin_ws/src/robot_nav/robots/xacros/omni_wheel.xacro (robot description, xacro)
@@ -22,5 +22,5 @@
      <origin xyz="0 0 0" rpy="0 0 0"/>
      <geometry>
-        <mesh filename="package://neo_simulation/robots/meshes/MPO-500-WHEEL.dae" scale="0.001 0.001 0.001"/>
+        <mesh filename="package://robot_nav/robots/meshes/MPO-500-WHEEL.dae" scale="0.001 0.001 0.001"/>
      </geometry>
     </visual>
@@ -28,5 +28,5 @@
      <origin xyz="0 0 0" rpy="0 1.57 1.57" />
      <geometry>
-        <!-- <mesh filename="package://neo_simulation/robots/meshes/MPO-500-WHEEL.dae" scale="0.001 0.001 0.001"/> -->
+        <!-- <mesh filename="package://robot_nav/robots/meshes/MPO-500-WHEEL.dae" scale="0.001 0.001 0.001"/> -->
        <!-- <cylinder radius="0.126" length="0.110"/> -->
       <sphere radius="0.117" />

File: catkin_ws/src/robot_nav/robots/xacros/sick_S300.xacro (robot description, xacro)
@@ -17,5 +17,5 @@
         <origin xyz="0 0 -0.12" rpy="-1.57 0 3.14" />
         <geometry>
-        <mesh filename="package://neo_simulation/robots/meshes/SICK-S300.dae" scale="0.001 0.001 0.001" />
+        <mesh filename="package://robot_nav/robots/meshes/SICK-S300.dae" scale="0.001 0.001 0.001" />
         </geometry>
       </visual>
@@ -23,5 +23,5 @@
         <origin xyz="0 0 -0.12" rpy="-1.57 0 3.14" />
         <geometry>
-        <mesh filename="package://neo_simulation/robots/meshes/SICK-S300.dae" scale="0.001 0.001 0.001" />
+        <mesh filename="package://robot_nav/robots/meshes/SICK-S300.dae" scale="0.001 0.001 0.001" />
         </geometry>
       </collision>

File: catkin_ws/src/robot_nav/robots/xacros/sick_laser.xacro (robot description, xacro)
@@ -18,5 +18,5 @@
       <origin xyz="0 0 -0.12" rpy="-1.57 0 3.14" />
         <geometry>
-        <mesh filename="package://neo_simulation/robots/meshes/SICK-S300.dae" scale="0.001 0.001 0.001" />
+        <mesh filename="package://robot_nav/robots/meshes/SICK-S300.dae" scale="0.001 0.001 0.001" />
         </geometry>
       </visual>
@@ -24,5 +24,5 @@
         <origin xyz="0 0 0" rpy="-1.57 0 3.14" />
         <geometry>
-        <mesh filename="package://neo_simulation/robots/meshes/SICK-S300.dae" scale="0.001 0.001 0.001" />
+        <mesh filename="package://robot_nav/robots/meshes/SICK-S300.dae" scale="0.001 0.001 0.001" />
         </geometry>
       </collision>
@@ -30,5 +30,5 @@
 <!--  <origin xyz="-0.0 0 -0.06" rpy="1.57 0 0" />
       <geometry>
-      <mesh filename="package://neo_simulation/robots/meshes/SICK-MICROSCAN3.dae" scale="0.001 0.001 0.001" />
+      <mesh filename="package://robot_nav/robots/meshes/SICK-MICROSCAN3.dae" scale="0.001 0.001 0.001" />
       </geometry>
       </visual>
@@ -36,5 +36,5 @@
  <origin xyz="-0.0 0 -0.06" rpy="1.57 0 0" />
       <geometry>
-        <mesh filename="package://neo_simulation/robots/meshes/SICK-MICROSCAN3.dae" scale="0.001 0.001 0.001" />
+        <mesh filename="package://robot_nav/robots/meshes/SICK-MICROSCAN3.dae" scale="0.001 0.001 0.001" />
         </geometry>
       </collision> -->

Commit message: parameter documentation

File: catkin_ws/src/robot_nav/robots/robot.urdf.xacro (robot description, xacro)
@@ -43,74 +43,6 @@
   </xacro:imu>
   <-->
-  <!--+++++++++++++++++++ Ultra Sonic ++++++++++++++++++++++++-->
-  <!-- Comment or uncomment based on your requirement -->
-  <!-- SENSOR 1 -->
-  <!-->
-  <xacro:us_sensor name="us_1" parent="base_link">
-    <origin xyz="0.100 0 0.500" rpy="0 3.14 3.14" />
-  </xacro:us_sensor>
-  <-->
-  <!-- SENSOR 2 -->
-  <!-- xacro:us_sensor name="us_2" parent="base_link">
-    <origin xyz="0.110 0 0.300" rpy="0 3.14 3.14" />
-  </xacro:us_sensor-->
-  <!-- SENSOR 3 -->
-  <!-- xacro:us_sensor name="us_3" parent="base_link">
-    <origin xyz="0.120 0 0.300" rpy="0 3.14 3.14" />
-  </xacro:us_sensor-->
-  <!-- SENSOR 4 -->
-  <!-- xacro:us_sensor name="us_4" parent="base_link">
-    <origin xyz="0.130 0 0.300" rpy="0 3.14 3.14" />
-  </xacro:us_sensor-->
-  <!-- SENSOR 5 -->
-  <!-- xacro:us_sensor name="us_5" parent="base_link">
-    <origin xyz="0.140 0 0.300" rpy="0 3.14 3.14" />
-  </xacro:us_sensor-->
-  <!-- SENSOR 6 -->
-  <!-- xacro:us_sensor name="us_6" parent="base_link">
-    <origin xyz="0.150 0 0.300" rpy="0 3.14 3.14" />
-  </xacro:us_sensor-->
-  <!-- SENSOR 7 -->
-  <!-- xacro:us_sensor name="us_7" parent="base_link">
-    <origin xyz="0.160 0 0.300" rpy="0 3.14 3.14" />
-  </xacro:us_sensor-->
-  <!-- SENSOR 8 -->
-  <!-- xacro:us_sensor name="us_8" parent="base_link">
-    <origin xyz="0.170 0 0.300" rpy="0 3.14 3.14" />
-  </xacro:us_sensor-->
-  <!-- SENSOR 9 -->
-  <!-- xacro:us_sensor name="us_9" parent="base_link">
-    <origin xyz="0.180 0 0.300" rpy="0 3.14 3.14" />
-  </xacro:us_sensor-->
-  <!-- SENSOR 10 -->
-  <!-- xacro:us_sensor name="us_10" parent="base_link">
-    <origin xyz="0.100 0 0.300" rpy="0 3.14 3.14" />
-  </xacro:us_sensor-->
-  <!-- SENSOR 11 -->
-  <!-- xacro:us_sensor name="us_11" parent="base_link">
-    <origin xyz="0.100 0 0.300" rpy="0 3.14 3.14" />
-  </xacro:us_sensor-->
-  <!-- SENSOR 12 -->
-  <!-- xacro:us_sensor name="us_12" parent="base_link">
-    <origin xyz="0.190 0 0.300" rpy="0 3.14 3.14" />
-  </xacro:us_sensor-->
-  <!-- SENSOR 13 -->
-  <!-- xacro:us_sensor name="us_13" parent="base_link">
-    <origin xyz="0.200 0 0.300" rpy="0 3.14 3.14" />
-  </xacro:us_sensor-->
-  <!-- SENSOR 14 -->
-  <!-- xacro:us_sensor name="us_14" parent="base_link">
-    <origin xyz="0.210 0 0.300" rpy="0 3.14 3.14" />
-  </xacro:us_sensor-->
-  <!-- SENSOR 15 -->
-  <!-- xacro:us_sensor name="us_15" parent="base_link">
-    <origin xyz="0.220 0 0.300" rpy="0 3.14 3.14" />
-  </xacro:us_sensor-->
-  <!-- SENSOR 16 -->
-  <!-- xacro:us_sensor name="us_16" parent="base_link">
-    <origin xyz="0.230 0 0.300" rpy="0 3.14 3.14" />
-  </xacro:us_sensor-->
-  <!--Camera  -->
-<!-- <xacro:camera name="camera" parent="base_link">
+  <!--Camera-->
+  <!-- <xacro:camera name="camera" parent="base_link">
     <origin xyz="0 0 0.38" rpy="0 0 0" />
   </xacro:camera> -->
